Commit message: or - update

File: urdf/ABot.urdf.xacro (robot description, xacro)
@@ -27,5 +27,5 @@
   </collision>
   </link>
-  <link name="box">
+   <link name="box">
   <inertial>
     <origin xyz="0 0 0" />
@@ -167,80 +167,95 @@
     <origin xyz="-0.15 0 0.025"/>
   </joint>
-  <!--link name="right_back_wheel">
-  <inertial>
-    <origin rpy="1.5707963267948966 0 0" xyz="0 0 0" />
-    <mass value="0.1" />
-    <inertia  ixx="0.01" ixy="0.0"  ixz="0.0"  iyy="0.01"  iyz="0.0"  izz="0.01" />
-  </inertial>
-  <visual>
-    <origin rpy="1.5707963267948966 0 0" xyz="0 0 0"/>
-    <geometry>
-      <cylinder length="0.05" radius="0.075"/>
-    </geometry>
-  </visual>
-  <collision>
-    <origin rpy="1.5707963267948966 0 0" xyz="0 0 0"/>
-    <geometry>
-      <cylinder length="0.05" radius="0.075"/>
-    </geometry>
-  </collision>
-  </link>
-  <gazebo reference="right_back_wheel">
-    <material>Gazebo/Black</material>
-  </gazebo>
-  <joint name="base_link_right_back_wheel" type="continuous">
-    <parent link="base_link"/>
-    <child link="right_back_wheel"/>
-    <axis xyz="0 1 0"/>
-    <origin xyz="-0.1 -0.15 0.075"/>
-  </joint>
-  <transmission name="T_base_link_right_back_wheel">
-    <type>transmission_interface/SimpleTransmission</type>
-    <actuator name="motor_3">
-      <mechanicalReduction>1</mechanicalReduction>
-      <hardwareInterface>hardware_interface/VelocityJointInterface</hardwareInterface>
-    </actuator>
-    <joint name="base_link_right_back_wheel">
-      <hardwareInterface>hardware_interface/VelocityJointInterface</hardwareInterface>
-    </joint>
-  </transmission>
-  <link name="left_back_wheel">
-  <inertial>
-    <origin rpy="1.5707963267948966 0 0" xyz="0 0 0" />
-    <mass value="0.1" />
-    <inertia  ixx="0.01" ixy="0.0"  ixz="0.0"  iyy="0.01"  iyz="0.0"  izz="0.01" />
-  </inertial>
-  <visual>
-    <origin rpy="1.5707963267948966 0 0" xyz="0 0 0"/>
-    <geometry>
-      <cylinder length="0.05" radius="0.075"/>
-    </geometry>
-  </visual>
-  <collision>
-    <origin rpy="1.5707963267948966 0 0" xyz="0 0 0"/>
-    <geometry>
-      <cylinder length="0.05" radius="0.075"/>
-    </geometry>
-  </collision>
-  </link>
-  <gazebo reference="left_back_wheel">
-    <material>Gazebo/Black</material>
-  </gazebo>
-  <joint name="base_link_left_back_wheel" type="continuous">
-    <parent link="base_link"/>
-    <child link="left_back_wheel"/>
-    <axis xyz="0 1 0"/>
-    <origin xyz="-0.1 0.15 0.075"/>
-  </joint>
-  <transmission name="T_base_link_left_back_wheel">
-    <type>transmission_interface/SimpleTransmission</type>
-    <actuator name="motor_4">
-      <mechanicalReduction>1</mechanicalReduction>
-      <hardwareInterface>hardware_interface/VelocityJointInterface</hardwareInterface>
-    </actuator>
-    <joint name="base_link_left_back_wheel">
-      <hardwareInterface>hardware_interface/VelocityJointInterface</hardwareInterface>
-    </joint>
-  </transmission-->
+<link name="camera_link1">
+    <collision>
+      <origin xyz="0 0 0" rpy="0 0 0"/>
+      <geometry>
+    <box size="0.01 0.01 0.01"/>
+      </geometry>
+    </collision>
+    <visual>
+      <origin xyz="0 0 0" rpy="0 0 0"/>
+      <geometry>
+    <box size="0.01 0.01 0.01"/>
+      </geometry>
+      <material name="red"/>
+    </visual>
+    <inertial>
+      <mass value="1e-5" />
+      <origin xyz="0 0 0" rpy="0 0 0"/>
+      <inertia ixx="1e-6" ixy="0" ixz="0" iyy="1e-6" iyz="0" izz="1e-6" />
+    </inertial>
+  </link>
+<joint name="hokuyo_joint" type="fixed">
+    <axis xyz="0 1 0" />
+    <origin xyz="0.15 0 0.2" rpy="0 0 0"/>
+    <parent link="base_link"/>
+    <child link="hokuyo_link"/>
+  </joint>
+  <!-- Hokuyo Laser -->
+  <link name="hokuyo_link">
+    <collision>
+      <origin xyz="0 0 0" rpy="0 0 0"/>
+      <geometry>
+    <box size="0.1 0.1 0.1"/>
+      </geometry>
+    </collision>
+    <visual>
+      <origin xyz="0 0 0" rpy="0 0 0"/>
+      <geometry>
+        <mesh filename="package://SLAM/urdf/hokuyo.dae"/>
+      </geometry>
+    </visual>
+    <inertial>
+      <mass value="1e-5" />
+      <origin xyz="0 0 0" rpy="0 0 0"/>
+      <inertia ixx="1e-6" ixy="0" ixz="0" iyy="1e-6" iyz="0" izz="1e-6" />
+    </inertial>
+  </link>
+<joint name="camera_joint1" type="fixed">
+    <axis xyz="0 1 0" />
+    <origin xyz="0.2 0 0.25" rpy="0 0 0"/>
+    <parent link="base_link"/>
+    <child link="camera_link1"/>
+  </joint>
+<gazebo reference="camera_link1">
+    <sensor type="camera" name="camera1">
+      <update_rate>30.0</update_rate>
+      <camera name="head">
+        <horizontal_fov>1.3962634</horizontal_fov>
+        <image>
+          <width>640</width>
+          <height>480</height>
+          <format>R8G8B8</format>
+        </image>
+        <clip>
+          <near>0.02</near>
+          <far>300</far>
+        </clip>
+        <noise>
+          <type>gaussian</type>
+          <!-- Noise is sampled independently per pixel on each frame.
+               That pixel's noise value is added to each of its color
+               channels, which at that point lie in the range [0,1]. -->
+          <mean>0.0</mean>
+          <stddev>0.007</stddev>
+        </noise>
+      </camera>
+      <plugin name="camera_controller" filename="libgazebo_ros_camera.so">
+        <alwaysOn>true</alwaysOn>
+        <updateRate>0.0</updateRate>
+        <cameraName>/camera</cameraName>
+        <imageTopicName>image_raw</imageTopicName>
+        <cameraInfoTopicName>camera_info</cameraInfoTopicName>
+        <frameName>camera_link1</frameName>
+        <hackBaseline>0.07</hackBaseline>
+        <distortionK1>0.0</distortionK1>
+        <distortionK2>0.0</distortionK2>
+        <distortionK3>0.0</distortionK3>
+        <distortionT1>0.0</distortionT1>
+        <distortionT2>0.0</distortionT2>
+      </plugin>
+    </sensor>
+  </gazebo>
 <gazebo>
   <plugin name="differential_drive_controller" filename="libgazebo_ros_diff_drive.so">
@@ -257,8 +272,43 @@
     <robotBaseFrame>base_link</robotBaseFrame>
     <publishWheelJointState>true</publishWheelJointState>
-    <enable_odom_tf>true</enable_odom_tf>
+    <enable_odom_tf>false</enable_odom_tf>
   </plugin>
 </gazebo>
-  <xacro:include filename="$(find SLAM)/urdf/hokuyo.xacro"/>
-  <xacro:laser name="base_laser" parent="base_link" xyz="0.225 0 0.2" rpy="0 0 0" meshes="package://gazebo_plugins/test/multi_robot_scenario/meshes/laser"/>
+ <gazebo reference="hokuyo_link">
+    <sensor type="gpu_ray" name="head_hokuyo_sensor">
+      <pose>0 0 0 0 0 0</pose>
+      <visualize>false</visualize>
+      <update_rate>5</update_rate>
+      <ray>
+        <scan>
+          <horizontal>
+            <samples>720</samples>
+            <resolution>1</resolution>
+            <min_angle>-1.570796</min_angle>
+            <max_angle>1.570796</max_angle>
+          </horizontal>
+        </scan>
+        <range>
+          <min>0.10</min>
+          <max>10.0</max>
+          <resolution>0.01</resolution>
+        </range>
+        <noise>
+          <type>gaussian</type>
+          <!-- Noise parameters based on published spec for Hokuyo laser
+               achieving "+-30mm" accuracy at range < 10m.  A mean of 0.0m and
+               stddev of 0.01m will put 99.7% of samples within 0.03m of the true
+               reading. -->
+          <mean>0.0</mean>
+          <stddev>0.01</stddev>
+        </noise>
+      </ray>
+      <plugin name="gazebo_ros_head_hokuyo_controller" filename="libgazebo_ros_gpu_laser.so">
+        <topicName>scan</topicName>
+        <frameName>hokuyo_link</frameName>
+      </plugin>
+    </sensor>
+  </gazebo>
+  <xacro:property name="hokuyo_link" value="0.05" />
+  <xacro:property name="camera_link1" value="0.05" />
 </robot>
